Commit message: nearly completed urdf, needs to be tested and absolutely needs a launch file

File: src/RoombaV2/constants.xacro (robot description, xacro)
@@ -12,3 +12,6 @@
     <xacro:property name="LEG_HEIGHT" value="0.5" />
     <xacro:property name="LEG_LENGTH" value="0.5" />
+    <xacro:property name="MASS" value="3" />
+    <xacro:property name="WHEEL_MASS" value="3" />
+    <xacro:property name="LEG_MASS" value="0.2" />
 </robot>

File: src/RoombaV2/roombav2.urdf.xacro (robot description, xacro)
@@ -3,151 +3,224 @@
     <xacro:include filename="constants.xacro" />
     <xacro:include filename="inertial_macros.xacro" />
+    <!-- defining the colors of your microver -->
     <material name="black">
-        <color rgba="0 0 0 1"/>
+        <color rgba="0 0 0 1" />
     </material>
     <material name="white">
-        <color rgba="1 1 1 1"/>
+        <color rgba="1 1 1 1" />
     </material>
     <material name="blue">
-        <color rgba="0.2 0.2 1 1"/>
+        <color rgba="0.2 0.2 1 1" />
     </material>
-    <!-- ####################### LINKS ########################## -->
-    <!-- the base link is in the middle of both back wheels -->
+    <!-- the base link located in the middle of the line between the center of both back wheels -->
     <link name="base_link">
     </link>
+                    <!-- ####################### JOINTS ########################## -->
+    <joint name="chassis_joint" type="fixed">
+        <origin xyz="0 0 0" rpy="0 0 0" />
+        <parent link="base_link" />
+        <child link="chassis" />
+    </joint>
+    <!-- WHEEL JOINTS -->
+    <joint name="front_left_wheel_joint" type="continuous">
+        <origin xyz="${LENGTH - LEG_LENGTH} ${((WIDTH/2) + LEG_WIDTH + (WHEEL_WIDTH/2))} 0" rpy="-${pi/2} 0 0" />
+        <parent link="base_link" />
+        <child link="front_left_wheel_link" />
+        <axis xyz="0 0 1"/>
+    </joint>
+    <joint name="front_right_wheel_joint" type="continuous">
+        <origin xyz="${LENGTH - LEG_LENGTH} ${-((WIDTH/2) + LEG_WIDTH + (WHEEL_WIDTH/2))} 0" rpy="${pi/2} 0 0" />
+        <parent link="base_link" />
+        <child link="front_right_wheel_link" />
+        <axis xyz="0 0 -1"/>
+    </joint>
+    <joint name="back_left_wheel_joint" type="continuous">
+        <origin xyz="0 ${((WIDTH/2) + LEG_WIDTH + (WHEEL_WIDTH/2))} 0" rpy="-${pi/2} 0 0" />
+        <parent link="base_link" />
+        <child link="back_left_wheel_link" />
+        <axis xyz="0 0 1"/>
+    </joint>
+    <joint name="back_right_wheel_joint" type="continuous">
+        <origin xyz="0 ${-((WIDTH/2) + LEG_WIDTH + (WHEEL_WIDTH/2))} 0" rpy="${pi/2} 0 0" />
+        <parent link="base_link" />
+        <child link="back_right_wheel_link" />
+        <axis xyz="0 0 -1"/>
+    </joint>
+    <!-- LEG JOINTS = FIXED -->
+    <joint name="back_left_leg_joint" type="fixed">
+        <origin xyz="0 ${((WIDTH/2)+(LEG_WIDTH/2))} ${LEG_HEIGHT/2}" rpy="0 0 0" />
+        <parent link="base_link" />
+        <child link="back_left_leg_link" />
+    </joint>
+    <joint name="back_right_leg_joint" type="fixed">
+        <origin xyz="0 ${-((WIDTH/2)+(LEG_WIDTH/2))} ${LEG_HEIGHT/2}" rpy="0 0 0" />
+        <parent link="base_link" />
+        <child link="back_right_leg_link" />
+    </joint>
+    <joint name="front_left_leg_joint" type="fixed">
+        <origin xyz="${LENGTH - LEG_LENGTH} ${((WIDTH/2)+(LEG_WIDTH/2))} ${LEG_HEIGHT/2}" rpy="0 0 0" />
+        <parent link="base_link" />
+        <child link="front_left_leg_link" />
+    </joint>
+    <joint name="front_right_leg_joint" type="fixed">
+        <origin xyz="${LENGTH - LEG_LENGTH} ${-((WIDTH/2)+(LEG_WIDTH/2))} ${LEG_HEIGHT/2}"
+            rpy="0 0 0" />
+        <parent link="base_link" />
+        <child link="front_right_leg_link" />
+    </joint>
+                    <!-- ####################### LINKS ########################## -->
     <link name="chassis">
         <visual>
             <geometry>
-                <box size="${LENGTH} ${WIDTH} ${HEIGHT}"/>
-            </geometry>
-            <material name="black"/>
-        </visual>
-        <collision>
-            <geometry>
-                <box size="${LENGTH} ${WIDTH} ${HEIGHT}"/>
-            </geometry>
-        </collision>
-    </link>
-                                    <!-- LEG LINKS -->
+                <box size="${LENGTH} ${WIDTH} ${HEIGHT}" />
+            </geometry>
+            <origin xyz="${LENGTH/2} 0 ${HEIGHT/2}" rpy="0 0 0"/>
+            <material name="black" />
+        </visual>
+        <collision>
+            <geometry>
+                <box size="${LENGTH} ${WIDTH} ${HEIGHT}" />
+            </geometry>
+            <origin xyz="${LENGTH/2} 0 ${HEIGHT/2}" rpy="0 0 0"/>
+        </collision>
+        <xacro:inertial_box mass="${MASS}" x="${LENGTH}" y="${WIDTH}" z="${HEIGHT}">
+            <origin xyz="${LENGTH/2} 0 ${HEIGHT/2}" rpy="0 0 0"/>
+        </xacro:inertial_box>
+    </link>
+                                        <!-- LEG LINKS -->
+    <!-- need to add inertias for the legs -->
     <link name="back_left_leg_link">
         <visual>
             <geometry>
-                <box size="${LEG_LENGTH} ${LEG_WIDTH} ${LEG_HEIGHT}"/>
-            </geometry>
-            <origin xyz="0 ${((WIDTH/2)+(LEG_WIDTH/2))} ${LEG_HEIGHT/2}"/>
-            <material name="black"/>
-        </visual>
+                <box size="${LEG_LENGTH} ${LEG_WIDTH} ${LEG_HEIGHT}" />
+            </geometry>
+            <origin xyz="0 ${((WIDTH/2)+(LEG_WIDTH/2))} ${LEG_HEIGHT/2}" />
+            <material name="black" />
+        </visual>
+        <collision>
+            <geometry>
+                <box size="${LEG_LENGTH} ${LEG_WIDTH} ${LEG_HEIGHT}" />
+            </geometry>
+            <origin xyz="0 ${((WIDTH/2)+(LEG_WIDTH/2))} ${LEG_HEIGHT/2}" />
+        </collision>
+        <xacro:inertial_box mass="${LEG_MASS}" x="${LEG_LENGTH}" y="${LEG_WIDTH}" z="${LEG_HEIGHT}">
+            <origin xyz="0 ${((WIDTH/2)+(LEG_WIDTH/2))} ${LEG_HEIGHT/2}" />
+        </xacro:inertial_box>
     </link>
     <link name="back_right_leg_link">
         <visual>
             <geometry>
-                <box size="${LEG_LENGTH} ${LEG_WIDTH} ${LEG_HEIGHT}"/>
-            </geometry>
-            <origin xyz="0 ${-((WIDTH/2)+(LEG_WIDTH/2))} ${LEG_HEIGHT/2}"/>
-            <material name="black"/>
-        </visual>
+                <box size="${LEG_LENGTH} ${LEG_WIDTH} ${LEG_HEIGHT}" />
+            </geometry>
+            <origin xyz="0 ${-((WIDTH/2)+(LEG_WIDTH/2))} ${LEG_HEIGHT/2}" />
+            <material name="black" />
+        </visual>
+        <collision>
+            <geometry>
+                <box size="${LEG_LENGTH} ${LEG_WIDTH} ${LEG_HEIGHT}" />
+            </geometry>
+            <origin xyz="0 ${-((WIDTH/2)+(LEG_WIDTH/2))} ${LEG_HEIGHT/2}" />
+        </collision>
+        <xacro:inertial_box mass="${LEG_MASS}" x="${LEG_LENGTH}" y="${LEG_WIDTH}" z="${LEG_HEIGHT}">
+            <origin xyz="0 ${-((WIDTH/2)+(LEG_WIDTH/2))} ${LEG_HEIGHT/2}" />
+        </xacro:inertial_box>
     </link>
     <link name="front_left_leg_link">
         <visual>
             <geometry>
-                <box size="${LEG_LENGTH} ${LEG_WIDTH} ${LEG_HEIGHT}"/>
-            </geometry>
-            <origin xyz="${LENGTH - LEG_LENGTH} ${((WIDTH/2)+(LEG_WIDTH/2))} ${LEG_HEIGHT/2}"/>
-            <material name="black"/>
-        </visual>
+                <box size="${LEG_LENGTH} ${LEG_WIDTH} ${LEG_HEIGHT}" />
+            </geometry>
+            <origin xyz="${LENGTH - LEG_LENGTH} ${((WIDTH/2)+(LEG_WIDTH/2))} ${LEG_HEIGHT/2}" />
+            <material name="black" />
+        </visual>
+        <collision>
+            <geometry>
+                <box size="${LEG_LENGTH} ${LEG_WIDTH} ${LEG_HEIGHT}" />
+            </geometry>
+            <origin xyz="${LENGTH - LEG_LENGTH} ${((WIDTH/2)+(LEG_WIDTH/2))} ${LEG_HEIGHT/2}" />
+        </collision>
+        <xacro:inertial_box mass="${LEG_MASS}" x="${LEG_LENGTH}" y="${LEG_WIDTH}" z="${LEG_HEIGHT}">
+            <origin xyz="${LENGTH - LEG_LENGTH} ${((WIDTH/2)+(LEG_WIDTH/2))} ${LEG_HEIGHT/2}" />
+        </xacro:inertial_box>
     </link>
     <link name="front_right_leg_link">
         <visual>
             <geometry>
-                <box size="${LEG_LENGTH} ${LEG_WIDTH} ${LEG_HEIGHT}"/>
-            </geometry>
-            <origin xyz="${LENGTH - LEG_LENGTH} ${-((WIDTH/2)+(LEG_WIDTH/2))} ${LEG_HEIGHT/2}"/>
-            <material name="black"/>
-        </visual>
-    </link>
-                                    <!-- WHEEL LINKS -->
+                <box size="${LEG_LENGTH} ${LEG_WIDTH} ${LEG_HEIGHT}" />
+            </geometry>
+            <origin xyz="${LENGTH - LEG_LENGTH} ${-((WIDTH/2)+(LEG_WIDTH/2))} ${LEG_HEIGHT/2}" />
+            <material name="black" />
+        </visual>
+        <collision>
+            <geometry>
+                <box size="${LEG_LENGTH} ${LEG_WIDTH} ${LEG_HEIGHT}" />
+            </geometry>
+            <origin xyz="${LENGTH - LEG_LENGTH} ${-((WIDTH/2)+(LEG_WIDTH/2))} ${LEG_HEIGHT/2}" />
+        </collision>
+        <xacro:inertial_box mass="${LEG_MASS}" x="${LEG_LENGTH}" y="${LEG_WIDTH}" z="${LEG_HEIGHT}">
+            <origin xyz="${LENGTH - LEG_LENGTH} ${-((WIDTH/2)+(LEG_WIDTH/2))} ${LEG_HEIGHT/2}" />
+        </xacro:inertial_box>
+    </link>
+                                        <!-- WHEEL LINKS -->
     <link name="front_left_wheel_link">
         <visual>
             <geometry>
-                <cylinder radius="${WHEEL_RADIUS}" length="${WHEEL_WIDTH}"/>
-            </geometry>
-            <material name="blue"/>
-        </visual>
-        <collision>
-            <geometry>
-                <cylinder radius="${WHEEL_RADIUS}" length="${WHEEL_WIDTH}"/>
-            </geometry>
-        </collision>
+                <cylinder radius="${WHEEL_RADIUS}" length="${WHEEL_WIDTH}" />
+            </geometry>
+            <material name="blue" />
+        </visual>
+        <collision>
+            <geometry>
+                <cylinder radius="${WHEEL_RADIUS}" length="${WHEEL_WIDTH}" />
+            </geometry>
+        </collision>
+        <xacro:inertial_cylinder mass="${WHEEL_MASS}" length="${WHEEL_WIDTH}" radius="${WHEEL_RADIUS}">
+            <origin xyz="0 0 0" rpy="0 0 0"/>
+        </xacro:inertial_cylinder>
     </link>
     <link name="front_right_wheel_link">
         <visual>
             <geometry>
-                <cylinder radius="${WHEEL_RADIUS}" length="${WHEEL_WIDTH}"/>
-            </geometry>
-        </visual>
-        <collision>
-            <geometry>
-                <cylinder radius="${WHEEL_RADIUS}" length="${WHEEL_WIDTH}"/>
-            </geometry>
-        </collision>
+                <cylinder radius="${WHEEL_RADIUS}" length="${WHEEL_WIDTH}" />
+            </geometry>
+        </visual>
+        <collision>
+            <geometry>
+                <cylinder radius="${WHEEL_RADIUS}" length="${WHEEL_WIDTH}" />
+            </geometry>
+        </collision>
+        <xacro:inertial_cylinder mass="${WHEEL_MASS}" length="${WHEEL_WIDTH}" radius="${WHEEL_RADIUS}">
+            <origin xyz="0 0 0" rpy="0 0 0"/>
+        </xacro:inertial_cylinder>
     </link>
     <link name="back_left_wheel_link">
         <visual>
             <geometry>
-                <cylinder radius="${WHEEL_RADIUS}" length="${WHEEL_WIDTH}"/>
-            </geometry>
-            <origin xyz="0 ${-((WIDTH/2) + WHEEL_WIDTH)} 0" rpy="0 0 0" />
-        </visual>
-        <collision>
-            <geometry>
-                <cylinder radius="${WHEEL_RADIUS}" length="${WHEEL_WIDTH}"/>
-            </geometry>
-        </collision>
+                <cylinder radius="${WHEEL_RADIUS}" length="${WHEEL_WIDTH}" />
+            </geometry>
+        </visual>
+        <collision>
+            <geometry>
+                <cylinder radius="${WHEEL_RADIUS}" length="${WHEEL_WIDTH}" />
+            </geometry>
+        </collision>
+        <xacro:inertial_cylinder mass="${WHEEL_MASS}" length="${WHEEL_WIDTH}" radius="${WHEEL_RADIUS}">
+            <origin xyz="0 0 0" rpy="0 0 0"/>
+        </xacro:inertial_cylinder>
     </link>
     <link name="back_right_wheel_link">
         <visual>
             <geometry>
-                <cylinder radius="${WHEEL_RADIUS}" length="${WHEEL_WIDTH}"/>
-            </geometry>
-            <origin xyz="0 ${-((WIDTH/2) + WHEEL_WIDTH)} 0" rpy="0 0 0" />
-        </visual>
-        <collision>
-            <geometry>
-                <cylinder radius="${WHEEL_RADIUS}" length="${WHEEL_WIDTH}"/>
-            </geometry>
-        </collision>
-    </link>
-    <!-- ####################### JOINTS ########################## -->
-    <joint name="chassis_joint" type="fixed">
-        <origin xyz="0 0 ${HEIGHT/2}" rpy="0 0 0" />
-        <parent link="base_link" />
-        <child link="chassis" />
-    <joint name="front_left_wheel_joint" type="continuous">
-        <!-- Add joint properties for the front left wheel -->
-        <!-- ... -->
-        <origin xyz="0 ${WIDTH/2} 0" rpy="0 0 0" />
-        <parent link="base_link" />
-        <child link="front_left_wheel_link" />
-    </joint>
-    <joint name="front_right_wheel_joint" type="continuous">
-        <!-- Add joint properties for the front left wheel -->
-        <!-- ... -->
-        <origin xyz="0 ${-WIDTH/2} 0" rpy="0 0 0" />
-        <parent link="base_link" />
-        <child link="front_left_wheel_link" />
-    </joint>
-    <joint name="back_left_wheel_joint" type="continuous">
-        <!-- Add joint properties for the front left wheel -->
-        <!-- ... -->
-        <origin xyz="0 ${-WIDTH/2} 0" rpy="0 0 0" />
-        <parent link="base_link" />
-        <child link="front_left_wheel_link" />
-    </joint>
-    <joint name="back_right_wheel_joint" type="continuous">
-        <!-- Add joint properties for the front left wheel -->
-        <!-- ... -->
-        <origin xyz="0 ${-WIDTH/2} 0" rpy="0 0 0" />
-        <parent link="base_link" />
-        <child link="front_left_wheel_link" />
-    </joint>
+                <cylinder radius="${WHEEL_RADIUS}" length="${WHEEL_WIDTH}" />
+            </geometry>
+        </visual>
+        <collision>
+            <geometry>
+                <cylinder radius="${WHEEL_RADIUS}" length="${WHEEL_WIDTH}" />
+            </geometry>
+        </collision>
+        <xacro:inertial_cylinder mass="${WHEEL_MASS}" length="${WHEEL_WIDTH}" radius="${WHEEL_RADIUS}">
+            <origin xyz="0 0 0" rpy="0 0 0"/>
+        </xacro:inertial_cylinder>
+    </link>
 </robot>
