Commit message: somewhat microver looking but need to fix wheels

File: src/microver/description/microver.urdf.xacro (robot description, xacro)
@@ -15,4 +15,11 @@
     <!-- the base link located in the middle of the line between the center of both back wheels -->
     <link name="base_link">
+        <visual>
+            <geometry>
+                <cylinder length="0.003" radius="0.003"/>
+            </geometry>
+            <origin xyz="0 0 0" rpy="0 0 0"/>
+            <material name="white" />
+        </visual>
     </link>
                     <!-- ####################### JOINTS ########################## -->
@@ -47,5 +54,5 @@
         <axis xyz="0 0 -1"/>
     </joint>
-    <!-- LEG JOINTS = FIXED -->
+                                <!-- LEG JOINTS = FIXED -->
     <joint name="back_left_leg_joint" type="fixed">
         <origin xyz="0 ${((WIDTH/2)+(LEG_WIDTH/2))} ${LEG_HEIGHT/2}" rpy="0 0 0" />
@@ -75,5 +82,5 @@
                 <box size="${LENGTH} ${WIDTH} ${HEIGHT}" />
             </geometry>
-            <origin xyz="${LENGTH/2} 0 ${HEIGHT/2}" rpy="0 0 0"/>
+            <origin xyz="${LENGTH/2} 0 ${LEG_HEIGHT - HEIGHT/2}" rpy="0 0 0"/>
             <material name="black" />
         </visual>
@@ -95,15 +102,13 @@
                 <box size="${LEG_LENGTH} ${LEG_WIDTH} ${LEG_HEIGHT}" />
             </geometry>
-            <origin xyz="0 ${((WIDTH/2)+(LEG_WIDTH/2))} ${LEG_HEIGHT/2}" />
-            <material name="black" />
-        </visual>
-        <collision>
-            <geometry>
-                <box size="${LEG_LENGTH} ${LEG_WIDTH} ${LEG_HEIGHT}" />
-            </geometry>
-            <origin xyz="0 ${((WIDTH/2)+(LEG_WIDTH/2))} ${LEG_HEIGHT/2}" />
-        </collision>
-        <xacro:inertial_box mass="${LEG_MASS}" x="${LEG_LENGTH}" y="${LEG_WIDTH}" z="${LEG_HEIGHT}">
-            <origin xyz="0 ${((WIDTH/2)+(LEG_WIDTH/2))} ${LEG_HEIGHT/2}" />
+            <material name="black" />
+        </visual>
+        <collision>
+            <geometry>
+                <box size="${LEG_LENGTH} ${LEG_WIDTH} ${LEG_HEIGHT}" />
+            </geometry>
+        </collision>
+        <xacro:inertial_box mass="${LEG_MASS}" x="${LEG_LENGTH}" y="${LEG_WIDTH}" z="${LEG_HEIGHT}">
+            <origin xyz="0 0 0" />
         </xacro:inertial_box>
     </link>
@@ -113,15 +118,13 @@
                 <box size="${LEG_LENGTH} ${LEG_WIDTH} ${LEG_HEIGHT}" />
             </geometry>
-            <origin xyz="0 ${-((WIDTH/2)+(LEG_WIDTH/2))} ${LEG_HEIGHT/2}" />
-            <material name="black" />
-        </visual>
-        <collision>
-            <geometry>
-                <box size="${LEG_LENGTH} ${LEG_WIDTH} ${LEG_HEIGHT}" />
-            </geometry>
-            <origin xyz="0 ${-((WIDTH/2)+(LEG_WIDTH/2))} ${LEG_HEIGHT/2}" />
-        </collision>
-        <xacro:inertial_box mass="${LEG_MASS}" x="${LEG_LENGTH}" y="${LEG_WIDTH}" z="${LEG_HEIGHT}">
-            <origin xyz="0 ${-((WIDTH/2)+(LEG_WIDTH/2))} ${LEG_HEIGHT/2}" />
+            <material name="black" />
+        </visual>
+        <collision>
+            <geometry>
+                <box size="${LEG_LENGTH} ${LEG_WIDTH} ${LEG_HEIGHT}" />
+            </geometry>
+        </collision>
+        <xacro:inertial_box mass="${LEG_MASS}" x="${LEG_LENGTH}" y="${LEG_WIDTH}" z="${LEG_HEIGHT}">
+            <origin xyz="0 0 0" />
         </xacro:inertial_box>
     </link>
@@ -131,15 +134,13 @@
                 <box size="${LEG_LENGTH} ${LEG_WIDTH} ${LEG_HEIGHT}" />
             </geometry>
-            <origin xyz="${LENGTH - LEG_LENGTH} ${((WIDTH/2)+(LEG_WIDTH/2))} ${LEG_HEIGHT/2}" />
-            <material name="black" />
-        </visual>
-        <collision>
-            <geometry>
-                <box size="${LEG_LENGTH} ${LEG_WIDTH} ${LEG_HEIGHT}" />
-            </geometry>
-            <origin xyz="${LENGTH - LEG_LENGTH} ${((WIDTH/2)+(LEG_WIDTH/2))} ${LEG_HEIGHT/2}" />
-        </collision>
-        <xacro:inertial_box mass="${LEG_MASS}" x="${LEG_LENGTH}" y="${LEG_WIDTH}" z="${LEG_HEIGHT}">
-            <origin xyz="${LENGTH - LEG_LENGTH} ${((WIDTH/2)+(LEG_WIDTH/2))} ${LEG_HEIGHT/2}" />
+            <material name="black" />
+        </visual>
+        <collision>
+            <geometry>
+                <box size="${LEG_LENGTH} ${LEG_WIDTH} ${LEG_HEIGHT}" />
+            </geometry>
+        </collision>
+        <xacro:inertial_box mass="${LEG_MASS}" x="${LEG_LENGTH}" y="${LEG_WIDTH}" z="${LEG_HEIGHT}">
+            <origin xyz="0 0 0" />
         </xacro:inertial_box>
     </link>
@@ -149,15 +150,13 @@
                 <box size="${LEG_LENGTH} ${LEG_WIDTH} ${LEG_HEIGHT}" />
             </geometry>
-            <origin xyz="${LENGTH - LEG_LENGTH} ${-((WIDTH/2)+(LEG_WIDTH/2))} ${LEG_HEIGHT/2}" />
-            <material name="black" />
-        </visual>
-        <collision>
-            <geometry>
-                <box size="${LEG_LENGTH} ${LEG_WIDTH} ${LEG_HEIGHT}" />
-            </geometry>
-            <origin xyz="${LENGTH - LEG_LENGTH} ${-((WIDTH/2)+(LEG_WIDTH/2))} ${LEG_HEIGHT/2}" />
-        </collision>
-        <xacro:inertial_box mass="${LEG_MASS}" x="${LEG_LENGTH}" y="${LEG_WIDTH}" z="${LEG_HEIGHT}">
-            <origin xyz="${LENGTH - LEG_LENGTH} ${-((WIDTH/2)+(LEG_WIDTH/2))} ${LEG_HEIGHT/2}" />
+            <material name="black" />
+        </visual>
+        <collision>
+            <geometry>
+                <box size="${LEG_LENGTH} ${LEG_WIDTH} ${LEG_HEIGHT}" />
+            </geometry>
+        </collision>
+        <xacro:inertial_box mass="${LEG_MASS}" x="${LEG_LENGTH}" y="${LEG_WIDTH}" z="${LEG_HEIGHT}">
+            <origin xyz="0 0 0" />
         </xacro:inertial_box>
     </link>
