Commit message: changed constants and rviz works but it looks like shit

File: src/microver/description/constants.xacro (robot description, xacro)
@@ -1,17 +1,18 @@
 <?xml version="1.0"?>
 <robot xmlns:xacro="http://ros.org/wiki/xacro">
-    <xacro:property name="MAX_SPEED" value="0.5" />
-    <xacro:property name="MIN_SPEED" value="0.1" />
-    <xacro:property name="WHEEL_RADIUS" value="0.15" />
-    <xacro:property name="WHEEL_WIDTH" value="0.15" />
+    <!-- speeds are in m/2 or rad/s, dimensions in m, weights in kg -->
+    <xacro:property name="MAX_SPEED" value="5.5" />
+    <xacro:property name="MIN_SPEED" value="0.0" />
+    <xacro:property name="WHEEL_RADIUS" value="0.04" />
+    <xacro:property name="WHEEL_WIDTH" value="0.1" />
     <xacro:property name="WHEELBASE" value="0.5" />
-    <xacro:property name="HEIGHT" value="0.5" />
-    <xacro:property name="LENGTH" value="0.5" />
-    <xacro:property name="WIDTH" value="0.5" />
-    <xacro:property name="LEG_WIDTH" value="0.5" />
-    <xacro:property name="LEG_HEIGHT" value="0.5" />
-    <xacro:property name="LEG_LENGTH" value="0.5" />
+    <xacro:property name="HEIGHT" value="0.05" />
+    <xacro:property name="LENGTH" value="0.3" />
+    <xacro:property name="WIDTH" value="0.15" />
+    <xacro:property name="LEG_WIDTH" value="0.03" />
+    <xacro:property name="LEG_HEIGHT" value="0.1" />
+    <xacro:property name="LEG_LENGTH" value="0.05" />
     <xacro:property name="MASS" value="3" />
-    <xacro:property name="WHEEL_MASS" value="3" />
-    <xacro:property name="LEG_MASS" value="0.2" />
+    <xacro:property name="WHEEL_MASS" value="0.3" />
+    <xacro:property name="LEG_MASS" value="0.1" />
 </robot>

Commit message: fixed delta x for the chassis, still needs wheels

File: src/microver/description/constants.xacro (robot description, xacro)
@@ -7,12 +7,12 @@
     <xacro:property name="WHEEL_WIDTH" value="0.1" />
     <xacro:property name="WHEELBASE" value="0.5" />
+    <xacro:property name="WHEEL_MASS" value="0.3" />
     <xacro:property name="HEIGHT" value="0.05" />
     <xacro:property name="LENGTH" value="0.3" />
     <xacro:property name="WIDTH" value="0.15" />
+    <xacro:property name="MASS" value="3" />
     <xacro:property name="LEG_WIDTH" value="0.03" />
     <xacro:property name="LEG_HEIGHT" value="0.1" />
     <xacro:property name="LEG_LENGTH" value="0.05" />
-    <xacro:property name="MASS" value="3" />
-    <xacro:property name="WHEEL_MASS" value="0.3" />
     <xacro:property name="LEG_MASS" value="0.1" />
 </robot>

File: src/microver/description/microver.urdf.xacro (robot description, xacro)
@@ -3,5 +3,4 @@
     <xacro:include filename="constants.xacro" />
     <xacro:include filename="inertial_macros.xacro" />
-    <!-- defining the colors of your microver -->
     <material name="black">
         <color rgba="0 0 0 1" />
@@ -82,5 +81,5 @@
                 <box size="${LENGTH} ${WIDTH} ${HEIGHT}" />
             </geometry>
-            <origin xyz="${LENGTH/2} 0 ${LEG_HEIGHT - HEIGHT/2}" rpy="0 0 0"/>
+            <origin xyz="${LENGTH/2 - LEG_LENGTH/2} 0 ${LEG_HEIGHT - HEIGHT/2}" rpy="0 0 0"/>
             <material name="black" />
         </visual>
@@ -89,8 +88,8 @@
                 <box size="${LENGTH} ${WIDTH} ${HEIGHT}" />
             </geometry>
-            <origin xyz="${LENGTH/2} 0 ${HEIGHT/2}" rpy="0 0 0"/>
+            <origin xyz="${LENGTH/2 - LEG_LENGTH/2} 0 ${LEG_HEIGHT - HEIGHT/2}" rpy="0 0 0"/>
         </collision>
         <xacro:inertial_box mass="${MASS}" x="${LENGTH}" y="${WIDTH}" z="${HEIGHT}">
-            <origin xyz="${LENGTH/2} 0 ${HEIGHT/2}" rpy="0 0 0"/>
+            <origin xyz="${LENGTH/2 - LEG_LENGTH/2} 0 ${LEG_HEIGHT - HEIGHT/2}" rpy="0 0 0"/>
         </xacro:inertial_box>
     </link>

Commit message: finished urdf model, need to add movement

File: src/microver/description/constants.xacro (robot description, xacro)
@@ -2,17 +2,17 @@
 <robot xmlns:xacro="http://ros.org/wiki/xacro">
     <!-- speeds are in m/2 or rad/s, dimensions in m, weights in kg -->
-    <xacro:property name="MAX_SPEED" value="5.5" />
-    <xacro:property name="MIN_SPEED" value="0.0" />
+    <xacro:property name="MAX_SPEED"    value="5.5"  />
+    <xacro:property name="MIN_SPEED"    value="0.0"  />
     <xacro:property name="WHEEL_RADIUS" value="0.04" />
-    <xacro:property name="WHEEL_WIDTH" value="0.1" />
-    <xacro:property name="WHEELBASE" value="0.5" />
-    <xacro:property name="WHEEL_MASS" value="0.3" />
-    <xacro:property name="HEIGHT" value="0.05" />
-    <xacro:property name="LENGTH" value="0.3" />
-    <xacro:property name="WIDTH" value="0.15" />
-    <xacro:property name="MASS" value="3" />
-    <xacro:property name="LEG_WIDTH" value="0.03" />
-    <xacro:property name="LEG_HEIGHT" value="0.1" />
-    <xacro:property name="LEG_LENGTH" value="0.05" />
-    <xacro:property name="LEG_MASS" value="0.1" />
+    <xacro:property name="WHEEL_WIDTH"  value="0.05"  />
+    <xacro:property name="WHEELBASE"    value="0.5"  />
+    <xacro:property name="WHEEL_MASS"   value="0.3"  />
+    <xacro:property name="HEIGHT"       value="0.05" />
+    <xacro:property name="LENGTH"       value="0.3"  />
+    <xacro:property name="WIDTH"        value="0.15" />
+    <xacro:property name="MASS"         value="3"    />
+    <xacro:property name="LEG_WIDTH"    value="0.03" />
+    <xacro:property name="LEG_HEIGHT"   value="0.1"  />
+    <xacro:property name="LEG_LENGTH"   value="0.05" />
+    <xacro:property name="LEG_MASS"     value="0.1"  />
 </robot>

File: src/microver/description/microver.urdf.xacro (robot description, xacro)
@@ -28,7 +28,7 @@
         <child link="chassis" />
     </joint>
-    <!-- WHEEL JOINTS -->
+                                        <!-- WHEEL JOINTS -->
     <joint name="front_left_wheel_joint" type="continuous">
-        <origin xyz="${LENGTH - LEG_LENGTH} ${((WIDTH/2) + LEG_WIDTH + (WHEEL_WIDTH/2))} 0" rpy="-${pi/2} 0 0" />
+        <origin xyz="${LENGTH - LEG_LENGTH} ${((WIDTH/2) + LEG_WIDTH + (WHEEL_WIDTH/2))} ${WHEEL_RADIUS}" rpy="-${pi/2} 0 0" />
         <parent link="base_link" />
         <child link="front_left_wheel_link" />
@@ -36,5 +36,5 @@
     </joint>
     <joint name="front_right_wheel_joint" type="continuous">
-        <origin xyz="${LENGTH - LEG_LENGTH} ${-((WIDTH/2) + LEG_WIDTH + (WHEEL_WIDTH/2))} 0" rpy="${pi/2} 0 0" />
+        <origin xyz="${LENGTH - LEG_LENGTH} ${-((WIDTH/2) + LEG_WIDTH + (WHEEL_WIDTH/2))} ${WHEEL_RADIUS}" rpy="${pi/2} 0 0" />
         <parent link="base_link" />
         <child link="front_right_wheel_link" />
@@ -42,5 +42,5 @@
     </joint>
     <joint name="back_left_wheel_joint" type="continuous">
-        <origin xyz="0 ${((WIDTH/2) + LEG_WIDTH + (WHEEL_WIDTH/2))} 0" rpy="-${pi/2} 0 0" />
+        <origin xyz="0 ${((WIDTH/2) + LEG_WIDTH + (WHEEL_WIDTH/2))} ${WHEEL_RADIUS}" rpy="-${pi/2} 0 0" />
         <parent link="base_link" />
         <child link="back_left_wheel_link" />
@@ -48,5 +48,5 @@
     </joint>
     <joint name="back_right_wheel_joint" type="continuous">
-        <origin xyz="0 ${-((WIDTH/2) + LEG_WIDTH + (WHEEL_WIDTH/2))} 0" rpy="${pi/2} 0 0" />
+        <origin xyz="0 ${-((WIDTH/2) + LEG_WIDTH + (WHEEL_WIDTH/2))} ${WHEEL_RADIUS}" rpy="${pi/2} 0 0" />
         <parent link="base_link" />
         <child link="back_right_wheel_link" />
@@ -55,20 +55,20 @@
                                 <!-- LEG JOINTS = FIXED -->
     <joint name="back_left_leg_joint" type="fixed">
-        <origin xyz="0 ${((WIDTH/2)+(LEG_WIDTH/2))} ${LEG_HEIGHT/2}" rpy="0 0 0" />
+        <origin xyz="0 ${((WIDTH/2)+(LEG_WIDTH/2))} ${LEG_HEIGHT/2 + WHEEL_RADIUS}" rpy="0 0 0" />
         <parent link="base_link" />
         <child link="back_left_leg_link" />
     </joint>
     <joint name="back_right_leg_joint" type="fixed">
-        <origin xyz="0 ${-((WIDTH/2)+(LEG_WIDTH/2))} ${LEG_HEIGHT/2}" rpy="0 0 0" />
+        <origin xyz="0 ${-((WIDTH/2)+(LEG_WIDTH/2))} ${LEG_HEIGHT/2 + WHEEL_RADIUS}" rpy="0 0 0" />
         <parent link="base_link" />
         <child link="back_right_leg_link" />
     </joint>
     <joint name="front_left_leg_joint" type="fixed">
-        <origin xyz="${LENGTH - LEG_LENGTH} ${((WIDTH/2)+(LEG_WIDTH/2))} ${LEG_HEIGHT/2}" rpy="0 0 0" />
+        <origin xyz="${LENGTH - LEG_LENGTH} ${((WIDTH/2)+(LEG_WIDTH/2))} ${LEG_HEIGHT/2 + WHEEL_RADIUS}" rpy="0 0 0" />
         <parent link="base_link" />
         <child link="front_left_leg_link" />
     </joint>
     <joint name="front_right_leg_joint" type="fixed">
-        <origin xyz="${LENGTH - LEG_LENGTH} ${-((WIDTH/2)+(LEG_WIDTH/2))} ${LEG_HEIGHT/2}"
+        <origin xyz="${LENGTH - LEG_LENGTH} ${-((WIDTH/2)+(LEG_WIDTH/2))} ${LEG_HEIGHT/2 + WHEEL_RADIUS}"
             rpy="0 0 0" />
         <parent link="base_link" />
@@ -81,5 +81,5 @@
                 <box size="${LENGTH} ${WIDTH} ${HEIGHT}" />
             </geometry>
-            <origin xyz="${LENGTH/2 - LEG_LENGTH/2} 0 ${LEG_HEIGHT - HEIGHT/2}" rpy="0 0 0"/>
+            <origin xyz="${LENGTH/2 - LEG_LENGTH/2} 0 ${LEG_HEIGHT - HEIGHT/2 + WHEEL_RADIUS}" rpy="0 0 0"/>
             <material name="black" />
         </visual>
@@ -88,8 +88,8 @@
                 <box size="${LENGTH} ${WIDTH} ${HEIGHT}" />
             </geometry>
-            <origin xyz="${LENGTH/2 - LEG_LENGTH/2} 0 ${LEG_HEIGHT - HEIGHT/2}" rpy="0 0 0"/>
+            <origin xyz="${LENGTH/2 - LEG_LENGTH/2} 0 ${LEG_HEIGHT - HEIGHT/2 + WHEEL_RADIUS}" rpy="0 0 0"/>
         </collision>
         <xacro:inertial_box mass="${MASS}" x="${LENGTH}" y="${WIDTH}" z="${HEIGHT}">
-            <origin xyz="${LENGTH/2 - LEG_LENGTH/2} 0 ${LEG_HEIGHT - HEIGHT/2}" rpy="0 0 0"/>
+            <origin xyz="${LENGTH/2 - LEG_LENGTH/2} 0 ${LEG_HEIGHT - HEIGHT/2 + WHEEL_RADIUS}" rpy="0 0 0"/>
         </xacro:inertial_box>
     </link>
@@ -174,5 +174,5 @@
         </collision>
         <xacro:inertial_cylinder mass="${WHEEL_MASS}" length="${WHEEL_WIDTH}" radius="${WHEEL_RADIUS}">
-            <origin xyz="0 0 0" rpy="0 0 0"/>
+            <origin xyz="0 0 0"/>
         </xacro:inertial_cylinder>
     </link>
@@ -182,12 +182,13 @@
                 <cylinder radius="${WHEEL_RADIUS}" length="${WHEEL_WIDTH}" />
             </geometry>
-        </visual>
-        <collision>
-            <geometry>
-                <cylinder radius="${WHEEL_RADIUS}" length="${WHEEL_WIDTH}" />
-            </geometry>
-        </collision>
-        <xacro:inertial_cylinder mass="${WHEEL_MASS}" length="${WHEEL_WIDTH}" radius="${WHEEL_RADIUS}">
-            <origin xyz="0 0 0" rpy="0 0 0"/>
+            <material name="blue" />
+        </visual>
+        <collision>
+            <geometry>
+                <cylinder radius="${WHEEL_RADIUS}" length="${WHEEL_WIDTH}" />
+            </geometry>
+        </collision>
+        <xacro:inertial_cylinder mass="${WHEEL_MASS}" length="${WHEEL_WIDTH}" radius="${WHEEL_RADIUS}">
+            <origin xyz="0 0 0"/>
         </xacro:inertial_cylinder>
     </link>
@@ -197,12 +198,13 @@
                 <cylinder radius="${WHEEL_RADIUS}" length="${WHEEL_WIDTH}" />
             </geometry>
-        </visual>
-        <collision>
-            <geometry>
-                <cylinder radius="${WHEEL_RADIUS}" length="${WHEEL_WIDTH}" />
-            </geometry>
-        </collision>
-        <xacro:inertial_cylinder mass="${WHEEL_MASS}" length="${WHEEL_WIDTH}" radius="${WHEEL_RADIUS}">
-            <origin xyz="0 0 0" rpy="0 0 0"/>
+            <material name="blue" />
+        </visual>
+        <collision>
+            <geometry>
+                <cylinder radius="${WHEEL_RADIUS}" length="${WHEEL_WIDTH}" />
+            </geometry>
+        </collision>
+        <xacro:inertial_cylinder mass="${WHEEL_MASS}" length="${WHEEL_WIDTH}" radius="${WHEEL_RADIUS}">
+            <origin xyz="0 0 0"/>
         </xacro:inertial_cylinder>
     </link>
@@ -212,12 +214,13 @@
                 <cylinder radius="${WHEEL_RADIUS}" length="${WHEEL_WIDTH}" />
             </geometry>
-        </visual>
-        <collision>
-            <geometry>
-                <cylinder radius="${WHEEL_RADIUS}" length="${WHEEL_WIDTH}" />
-            </geometry>
-        </collision>
-        <xacro:inertial_cylinder mass="${WHEEL_MASS}" length="${WHEEL_WIDTH}" radius="${WHEEL_RADIUS}">
-            <origin xyz="0 0 0" rpy="0 0 0"/>
+            <material name="blue" />
+        </visual>
+        <collision>
+            <geometry>
+                <cylinder radius="${WHEEL_RADIUS}" length="${WHEEL_WIDTH}" />
+            </geometry>
+        </collision>
+        <xacro:inertial_cylinder mass="${WHEEL_MASS}" length="${WHEEL_WIDTH}" radius="${WHEEL_RADIUS}">
+            <origin xyz="0 0 0"/>
         </xacro:inertial_cylinder>
     </link>

Commit message: added arduino files

File: src/microver/description/constants.xacro (robot description, xacro)
@@ -7,5 +7,5 @@
     <xacro:property name="WHEEL_WIDTH"  value="0.05"  />
     <xacro:property name="WHEELBASE"    value="0.5"  />
-    <xacro:property name="WHEEL_MASS"   value="0.3"  />
+    <xacro:property name="WHEEL_MASS"   value="0.45"  />
     <xacro:property name="HEIGHT"       value="0.05" />
     <xacro:property name="LENGTH"       value="0.3"  />
@@ -16,5 +16,5 @@
     <xacro:property name="LEG_LENGTH"   value="0.05" />
     <xacro:property name="LEG_MASS"     value="0.1"  />
-    <xacro:property name="MU1"     value="0.1"  />
-    <xacro:property name="MU2"     value="0.1"  />
+    <xacro:property name="MU1"     value="0.3"  />
+    <xacro:property name="MU2"     value="0.3"  />
 </robot>
