Commit message: somewhat working simulation, need to fix movement inputs

File: install/microver/share/microver/description/gazebo_control.xacro (robot description, xacro)
@@ -1 +1 @@
-/home/arno/microver_ws/src/microver/description/gazebo_control.xacro
+/home/arno/BasestationRoombaV3/src/microver/description/gazebo_control.xacro

File: src/microver/description/constants.xacro (robot description, xacro)
@@ -16,3 +16,5 @@
     <xacro:property name="LEG_LENGTH"   value="0.05" />
     <xacro:property name="LEG_MASS"     value="0.1"  />
+    <xacro:property name="MU1"     value="0.1"  />
+    <xacro:property name="MU2"     value="0.1"  />
 </robot>

File: src/microver/description/microver.urdf.xacro (robot description, xacro)
@@ -3,4 +3,5 @@
     <xacro:include filename="constants.xacro" />
     <xacro:include filename="inertial_macros.xacro" />
+    <xacro:include filename="gazebo_control.xacro" />
     <material name="black">
         <color rgba="0 0 0 1" />
@@ -11,4 +12,7 @@
     <material name="blue">
         <color rgba="0.2 0.2 1 1" />
+    </material>
+    <material name="purple">
+        <color rgba="0.62 0.12 0.94 1" />
     </material>
     <!-- the base link located in the middle of the line between the center of both back wheels -->
@@ -34,4 +38,6 @@
         <child link="front_left_wheel_link" />
         <axis xyz="0 0 1"/>
+        <limit effort="100" velocity="100"/>
+        <dynamics damping="0.1" friction="0.1"/>
     </joint>
     <joint name="front_right_wheel_joint" type="continuous">
@@ -40,4 +46,6 @@
         <child link="front_right_wheel_link" />
         <axis xyz="0 0 -1"/>
+        <limit effort="100" velocity="100"/>
+        <dynamics damping="0.1" friction="0.1"/>
     </joint>
     <joint name="back_left_wheel_joint" type="continuous">
@@ -46,4 +54,6 @@
         <child link="back_left_wheel_link" />
         <axis xyz="0 0 1"/>
+        <limit effort="100" velocity="100"/>
+        <dynamics damping="0.1" friction="0.1"/>
     </joint>
     <joint name="back_right_wheel_joint" type="continuous">
@@ -52,4 +62,6 @@
         <child link="back_right_wheel_link" />
         <axis xyz="0 0 -1"/>
+        <limit effort="100" velocity="100"/>
+        <dynamics damping="0.1" friction="0.1"/>
     </joint>
                                 <!-- LEG JOINTS = FIXED -->
@@ -166,5 +178,5 @@
                 <cylinder radius="${WHEEL_RADIUS}" length="${WHEEL_WIDTH}" />
             </geometry>
-            <material name="blue" />
+            <material name="purple" />
         </visual>
         <collision>
@@ -182,5 +194,5 @@
                 <cylinder radius="${WHEEL_RADIUS}" length="${WHEEL_WIDTH}" />
             </geometry>
-            <material name="blue" />
+            <material name="purple" />
         </visual>
         <collision>
@@ -198,5 +210,5 @@
                 <cylinder radius="${WHEEL_RADIUS}" length="${WHEEL_WIDTH}" />
             </geometry>
-            <material name="blue" />
+            <material name="purple" />
         </visual>
         <collision>
@@ -214,14 +226,50 @@
                 <cylinder radius="${WHEEL_RADIUS}" length="${WHEEL_WIDTH}" />
             </geometry>
-            <material name="blue" />
-        </visual>
-        <collision>
-            <geometry>
-                <cylinder radius="${WHEEL_RADIUS}" length="${WHEEL_WIDTH}" />
-            </geometry>
-        </collision>
-        <xacro:inertial_cylinder mass="${WHEEL_MASS}" length="${WHEEL_WIDTH}" radius="${WHEEL_RADIUS}">
-            <origin xyz="0 0 0"/>
-        </xacro:inertial_cylinder>
-    </link>
+            <material name="purple" />
+        </visual>
+        <collision>
+            <geometry>
+                <cylinder radius="${WHEEL_RADIUS}" length="${WHEEL_WIDTH}" />
+            </geometry>
+        </collision>
+        <xacro:inertial_cylinder mass="${WHEEL_MASS}" length="${WHEEL_WIDTH}" radius="${WHEEL_RADIUS}">
+            <origin xyz="0 0 0"/>
+        </xacro:inertial_cylinder>
+    </link>
+                                                <!-- Gazebo -->
+    <gazebo reference="chassis">
+        <material>Gazebo/Black</material>
+    </gazebo>
+    <gazebo reference="back_left_leg_link">
+        <material>Gazebo/Black</material>
+    </gazebo>
+    <gazebo reference="back_right_leg_link">
+        <material>Gazebo/Black</material>
+    </gazebo>
+    <gazebo reference="front_left_leg_link">
+        <material>Gazebo/Black</material>
+    </gazebo>
+    <gazebo reference="front_right_leg_link">
+        <material>Gazebo/Black</material>
+    </gazebo>
+    <gazebo reference="front_left_wheel_link">
+        <material>Gazebo/Purple</material>
+        <mu1 value="${MU1}" />
+        <mu2 value="${MU2}" />
+    </gazebo>
+    <gazebo reference="front_right_wheel_link">
+        <material>Gazebo/Purple</material>
+        <mu1 value="${MU1}" />
+        <mu2 value="${MU2}" />
+    </gazebo>
+    <gazebo reference="back_left_wheel_link">
+        <material>Gazebo/Purple</material>
+        <mu1 value="${MU1}" />
+        <mu2 value="${MU2}" />
+    </gazebo>
+    <gazebo reference="back_right_wheel_link">
+        <material>Gazebo/Purple</material>
+        <mu1 value="${MU1}" />
+        <mu2 value="${MU2}" />
+    </gazebo>
 </robot>
