Commit message: uhhh dunno ngl, i just came back from my holidays and this stuff wasn't pushed yet

File: install/microver/share/microver/description/constants.xacro (robot description, xacro)
@@ -1 +1,20 @@
-/home/arno/BasestationRoombaV3/src/microver/description/constants.xacro
+<?xml version="1.0"?>
+<robot xmlns:xacro="http://ros.org/wiki/xacro">
+    <!-- speeds are in m/2 or rad/s, dimensions in m, weights in kg -->
+    <xacro:property name="MAX_SPEED"    value="5.5"  />
+    <xacro:property name="MIN_SPEED"    value="0.0"  />
+    <xacro:property name="WHEEL_RADIUS" value="0.04" />
+    <xacro:property name="WHEEL_WIDTH"  value="0.05"  />
+    <xacro:property name="WHEELBASE"    value="0.5"  />
+    <xacro:property name="WHEEL_MASS"   value="0.45"  />
+    <xacro:property name="HEIGHT"       value="0.05" />
+    <xacro:property name="LENGTH"       value="0.3"  />
+    <xacro:property name="WIDTH"        value="0.15" />
+    <xacro:property name="MASS"         value="3"    />
+    <xacro:property name="LEG_WIDTH"    value="0.03" />
+    <xacro:property name="LEG_HEIGHT"   value="0.1"  />
+    <xacro:property name="LEG_LENGTH"   value="0.05" />
+    <xacro:property name="LEG_MASS"     value="0.1"  />
+    <xacro:property name="MU1"     value="0.3"  />
+    <xacro:property name="MU2"     value="0.3"  />
+</robot>

File: install/microver/share/microver/description/gazebo_control.xacro (robot description, xacro)
@@ -1 +1,25 @@
-/home/arno/BasestationRoombaV3/src/microver/description/gazebo_control.xacro
+<?xml version="1.0"?>
+<robot xmlns:xacro="http://ros.org/wiki/xacro" name="microver">
+    <!-- Controller for the 4 wheeled differential drive microver inchallah-->
+    <gazebo>
+        <plugin name="skid_steer_drive" filename="libgazebo_ros_diff_drive.so">
+            <num_wheel_pairs>2</num_wheel_pairs>
+            <left_joint>front_left_wheel_joint</left_joint>
+            <right_joint>front_right_wheel_joint</right_joint>
+            <left_joint>back_left_wheel_joint</left_joint>
+            <right_joint>back_right_wheel_joint</right_joint>
+            <wheel_separation>${WIDTH + (2*LEG_WIDTH) + WHEEL_WIDTH}</wheel_separation>
+            <!-- <wheel_separation>${WIDTH + (2*LEG_WIDTH) + WHEEL_WIDTH}</wheel_separation> -->
+            <wheel_diameter>${2*WHEEL_RADIUS}</wheel_diameter>
+            <!-- <wheel_diameter>${2*WHEEL_RADIUS}</wheel_diameter> -->
+            <max_wheel_torque>5</max_wheel_torque>
+            <max_wheel_acceleration>5.0</max_wheel_acceleration>
+            <!-- output -->
+            <publish_odom>true</publish_odom>
+            <publish_odom_tf>true</publish_odom_tf>
+            <publish_wheel_tf>true</publish_wheel_tf>
+            <odometry_frame>odom</odometry_frame>
+            <robot_base_frame>base_link</robot_base_frame>
+        </plugin>
+    </gazebo>
+</robot>

File: install/microver/share/microver/description/inertial_macros.xacro (robot description, xacro)
@@ -1 +1,33 @@
-/home/arno/BasestationRoombaV3/src/microver/description/inertial_macros.xacro
+<?xml version="1.0"?>
+<robot xmlns:xacro="http://www.ros.org/wiki/xacro" >
+    <!-- ALL CREDITS GO TO JOSH NEWANS OF ARTICULATED ROBOTICS -->
+    <!-- Specify some standard inertial calculations https://en.wikipedia.org/wiki/List_of_moments_of_inertia -->
+    <!-- These make use of xacro's mathematical functionality -->
+    <xacro:macro name="inertial_sphere" params="mass radius *origin">
+        <inertial>
+            <xacro:insert_block name="origin"/>
+            <mass value="${mass}" />
+            <inertia ixx="${(2/5) * mass * (radius*radius)}" ixy="0.0" ixz="0.0"
+                    iyy="${(2/5) * mass * (radius*radius)}" iyz="0.0"
+                    izz="${(2/5) * mass * (radius*radius)}" />
+        </inertial>
+    </xacro:macro>
+    <xacro:macro name="inertial_box" params="mass x y z *origin">
+        <inertial>
+            <xacro:insert_block name="origin"/>
+            <mass value="${mass}" />
+            <inertia ixx="${(1/12) * mass * (y*y+z*z)}" ixy="0.0" ixz="0.0"
+                    iyy="${(1/12) * mass * (x*x+z*z)}" iyz="0.0"
+                    izz="${(1/12) * mass * (x*x+y*y)}" />
+        </inertial>
+    </xacro:macro>
+    <xacro:macro name="inertial_cylinder" params="mass length radius *origin">
+        <inertial>
+            <xacro:insert_block name="origin"/>
+            <mass value="${mass}" />
+            <inertia ixx="${(1/12) * mass * (3*radius*radius + length*length)}" ixy="0.0" ixz="0.0"
+                    iyy="${(1/12) * mass * (3*radius*radius + length*length)}" iyz="0.0"
+                    izz="${(1/2) * mass * (radius*radius)}" />
+        </inertial>
+    </xacro:macro>
+</robot>

File: install/microver/share/microver/description/microver.urdf.xacro (robot description, xacro)
@@ -1 +1,275 @@
-/home/arno/BasestationRoombaV3/src/microver/description/microver.urdf.xacro
+<?xml version="1.0"?>
+<robot xmlns:xacro="http://ros.org/wiki/xacro" name="microver">
+    <xacro:include filename="constants.xacro" />
+    <xacro:include filename="inertial_macros.xacro" />
+    <xacro:include filename="gazebo_control.xacro" />
+    <material name="black">
+        <color rgba="0 0 0 1" />
+    </material>
+    <material name="white">
+        <color rgba="1 1 1 1" />
+    </material>
+    <material name="blue">
+        <color rgba="0.2 0.2 1 1" />
+    </material>
+    <material name="purple">
+        <color rgba="0.62 0.12 0.94 1" />
+    </material>
+    <!-- the base link located in the middle of the line between the center of both back wheels -->
+    <link name="base_link">
+        <visual>
+            <geometry>
+                <cylinder length="0.003" radius="0.003"/>
+            </geometry>
+            <origin xyz="0 0 0" rpy="0 0 0"/>
+            <material name="white" />
+        </visual>
+    </link>
+                    <!-- ####################### JOINTS ########################## -->
+    <joint name="chassis_joint" type="fixed">
+        <origin xyz="0 0 0" rpy="0 0 0" />
+        <parent link="base_link" />
+        <child link="chassis" />
+    </joint>
+                                        <!-- WHEEL JOINTS -->
+    <joint name="front_left_wheel_joint" type="continuous">
+        <origin xyz="${LENGTH - LEG_LENGTH} ${((WIDTH/2) + LEG_WIDTH + (WHEEL_WIDTH/2))} ${WHEEL_RADIUS}" rpy="-${pi/2} 0 0" />
+        <parent link="base_link" />
+        <child link="front_left_wheel_link" />
+        <axis xyz="0 0 1"/>
+        <limit effort="100" velocity="100"/>
+        <dynamics damping="0.1" friction="0.1"/>
+    </joint>
+    <joint name="front_right_wheel_joint" type="continuous">
+        <origin xyz="${LENGTH - LEG_LENGTH} ${-((WIDTH/2) + LEG_WIDTH + (WHEEL_WIDTH/2))} ${WHEEL_RADIUS}" rpy="${pi/2} 0 0" />
+        <parent link="base_link" />
+        <child link="front_right_wheel_link" />
+        <axis xyz="0 0 -1"/>
+        <limit effort="100" velocity="100"/>
+        <dynamics damping="0.1" friction="0.1"/>
+    </joint>
+    <joint name="back_left_wheel_joint" type="continuous">
+        <origin xyz="0 ${((WIDTH/2) + LEG_WIDTH + (WHEEL_WIDTH/2))} ${WHEEL_RADIUS}" rpy="-${pi/2} 0 0" />
+        <parent link="base_link" />
+        <child link="back_left_wheel_link" />
+        <axis xyz="0 0 1"/>
+        <limit effort="100" velocity="100"/>
+        <dynamics damping="0.1" friction="0.1"/>
+    </joint>
+    <joint name="back_right_wheel_joint" type="continuous">
+        <origin xyz="0 ${-((WIDTH/2) + LEG_WIDTH + (WHEEL_WIDTH/2))} ${WHEEL_RADIUS}" rpy="${pi/2} 0 0" />
+        <parent link="base_link" />
+        <child link="back_right_wheel_link" />
+        <axis xyz="0 0 -1"/>
+        <limit effort="100" velocity="100"/>
+        <dynamics damping="0.1" friction="0.1"/>
+    </joint>
+                                <!-- LEG JOINTS = FIXED -->
+    <joint name="back_left_leg_joint" type="fixed">
+        <origin xyz="0 ${((WIDTH/2)+(LEG_WIDTH/2))} ${LEG_HEIGHT/2 + WHEEL_RADIUS}" rpy="0 0 0" />
+        <parent link="base_link" />
+        <child link="back_left_leg_link" />
+    </joint>
+    <joint name="back_right_leg_joint" type="fixed">
+        <origin xyz="0 ${-((WIDTH/2)+(LEG_WIDTH/2))} ${LEG_HEIGHT/2 + WHEEL_RADIUS}" rpy="0 0 0" />
+        <parent link="base_link" />
+        <child link="back_right_leg_link" />
+    </joint>
+    <joint name="front_left_leg_joint" type="fixed">
+        <origin xyz="${LENGTH - LEG_LENGTH} ${((WIDTH/2)+(LEG_WIDTH/2))} ${LEG_HEIGHT/2 + WHEEL_RADIUS}" rpy="0 0 0" />
+        <parent link="base_link" />
+        <child link="front_left_leg_link" />
+    </joint>
+    <joint name="front_right_leg_joint" type="fixed">
+        <origin xyz="${LENGTH - LEG_LENGTH} ${-((WIDTH/2)+(LEG_WIDTH/2))} ${LEG_HEIGHT/2 + WHEEL_RADIUS}"
+            rpy="0 0 0" />
+        <parent link="base_link" />
+        <child link="front_right_leg_link" />
+    </joint>
+                    <!-- ####################### LINKS ########################## -->
+    <link name="chassis">
+        <visual>
+            <geometry>
+                <box size="${LENGTH} ${WIDTH} ${HEIGHT}" />
+            </geometry>
+            <origin xyz="${LENGTH/2 - LEG_LENGTH/2} 0 ${LEG_HEIGHT - HEIGHT/2 + WHEEL_RADIUS}" rpy="0 0 0"/>
+            <material name="black" />
+        </visual>
+        <collision>
+            <geometry>
+                <box size="${LENGTH} ${WIDTH} ${HEIGHT}" />
+            </geometry>
+            <origin xyz="${LENGTH/2 - LEG_LENGTH/2} 0 ${LEG_HEIGHT - HEIGHT/2 + WHEEL_RADIUS}" rpy="0 0 0"/>
+        </collision>
+        <xacro:inertial_box mass="${MASS}" x="${LENGTH}" y="${WIDTH}" z="${HEIGHT}">
+            <origin xyz="${LENGTH/2 - LEG_LENGTH/2} 0 ${LEG_HEIGHT - HEIGHT/2 + WHEEL_RADIUS}" rpy="0 0 0"/>
+        </xacro:inertial_box>
+    </link>
+                                        <!-- LEG LINKS -->
+    <!-- need to add inertias for the legs -->
+    <link name="back_left_leg_link">
+        <visual>
+            <geometry>
+                <box size="${LEG_LENGTH} ${LEG_WIDTH} ${LEG_HEIGHT}" />
+            </geometry>
+            <material name="black" />
+        </visual>
+        <collision>
+            <geometry>
+                <box size="${LEG_LENGTH} ${LEG_WIDTH} ${LEG_HEIGHT}" />
+            </geometry>
+        </collision>
+        <xacro:inertial_box mass="${LEG_MASS}" x="${LEG_LENGTH}" y="${LEG_WIDTH}" z="${LEG_HEIGHT}">
+            <origin xyz="0 0 0" />
+        </xacro:inertial_box>
+    </link>
+    <link name="back_right_leg_link">
+        <visual>
+            <geometry>
+                <box size="${LEG_LENGTH} ${LEG_WIDTH} ${LEG_HEIGHT}" />
+            </geometry>
+            <material name="black" />
+        </visual>
+        <collision>
+            <geometry>
+                <box size="${LEG_LENGTH} ${LEG_WIDTH} ${LEG_HEIGHT}" />
+            </geometry>
+        </collision>
+        <xacro:inertial_box mass="${LEG_MASS}" x="${LEG_LENGTH}" y="${LEG_WIDTH}" z="${LEG_HEIGHT}">
+            <origin xyz="0 0 0" />
+        </xacro:inertial_box>
+    </link>
+    <link name="front_left_leg_link">
+        <visual>
+            <geometry>
+                <box size="${LEG_LENGTH} ${LEG_WIDTH} ${LEG_HEIGHT}" />
+            </geometry>
+            <material name="black" />
+        </visual>
+        <collision>
+            <geometry>
+                <box size="${LEG_LENGTH} ${LEG_WIDTH} ${LEG_HEIGHT}" />
+            </geometry>
+        </collision>
+        <xacro:inertial_box mass="${LEG_MASS}" x="${LEG_LENGTH}" y="${LEG_WIDTH}" z="${LEG_HEIGHT}">
+            <origin xyz="0 0 0" />
+        </xacro:inertial_box>
+    </link>
+    <link name="front_right_leg_link">
+        <visual>
+            <geometry>
+                <box size="${LEG_LENGTH} ${LEG_WIDTH} ${LEG_HEIGHT}" />
+            </geometry>
+            <material name="black" />
+        </visual>
+        <collision>
+            <geometry>
+                <box size="${LEG_LENGTH} ${LEG_WIDTH} ${LEG_HEIGHT}" />
+            </geometry>
+        </collision>
+        <xacro:inertial_box mass="${LEG_MASS}" x="${LEG_LENGTH}" y="${LEG_WIDTH}" z="${LEG_HEIGHT}">
+            <origin xyz="0 0 0" />
+        </xacro:inertial_box>
+    </link>
+                                        <!-- WHEEL LINKS -->
+    <link name="front_left_wheel_link">
+        <visual>
+            <geometry>
+                <cylinder radius="${WHEEL_RADIUS}" length="${WHEEL_WIDTH}" />
+            </geometry>
+            <material name="purple" />
+        </visual>
+        <collision>
+            <geometry>
+                <cylinder radius="${WHEEL_RADIUS}" length="${WHEEL_WIDTH}" />
+            </geometry>
+        </collision>
+        <xacro:inertial_cylinder mass="${WHEEL_MASS}" length="${WHEEL_WIDTH}" radius="${WHEEL_RADIUS}">
+            <origin xyz="0 0 0"/>
+        </xacro:inertial_cylinder>
+    </link>
+    <link name="front_right_wheel_link">
+        <visual>
+            <geometry>
+                <cylinder radius="${WHEEL_RADIUS}" length="${WHEEL_WIDTH}" />
+            </geometry>
+            <material name="purple" />
+        </visual>
+        <collision>
+            <geometry>
+                <cylinder radius="${WHEEL_RADIUS}" length="${WHEEL_WIDTH}" />
+            </geometry>
+        </collision>
+        <xacro:inertial_cylinder mass="${WHEEL_MASS}" length="${WHEEL_WIDTH}" radius="${WHEEL_RADIUS}">
+            <origin xyz="0 0 0"/>
+        </xacro:inertial_cylinder>
+    </link>
+    <link name="back_left_wheel_link">
+        <visual>
+            <geometry>
+                <cylinder radius="${WHEEL_RADIUS}" length="${WHEEL_WIDTH}" />
+            </geometry>
+            <material name="purple" />
+        </visual>
+        <collision>
+            <geometry>
+                <cylinder radius="${WHEEL_RADIUS}" length="${WHEEL_WIDTH}" />
+            </geometry>
+        </collision>
+        <xacro:inertial_cylinder mass="${WHEEL_MASS}" length="${WHEEL_WIDTH}" radius="${WHEEL_RADIUS}">
+            <origin xyz="0 0 0"/>
+        </xacro:inertial_cylinder>
+    </link>
+    <link name="back_right_wheel_link">
+        <visual>
+            <geometry>
+                <cylinder radius="${WHEEL_RADIUS}" length="${WHEEL_WIDTH}" />
+            </geometry>
+            <material name="purple" />
+        </visual>
+        <collision>
+            <geometry>
+                <cylinder radius="${WHEEL_RADIUS}" length="${WHEEL_WIDTH}" />
+            </geometry>
+        </collision>
+        <xacro:inertial_cylinder mass="${WHEEL_MASS}" length="${WHEEL_WIDTH}" radius="${WHEEL_RADIUS}">
+            <origin xyz="0 0 0"/>
+        </xacro:inertial_cylinder>
+    </link>
+                                                <!-- Gazebo -->
+    <gazebo reference="chassis">
+        <material>Gazebo/Black</material>
+    </gazebo>
+    <gazebo reference="back_left_leg_link">
+        <material>Gazebo/Black</material>
+    </gazebo>
+    <gazebo reference="back_right_leg_link">
+        <material>Gazebo/Black</material>
+    </gazebo>
+    <gazebo reference="front_left_leg_link">
+        <material>Gazebo/Black</material>
+    </gazebo>
+    <gazebo reference="front_right_leg_link">
+        <material>Gazebo/Black</material>
+    </gazebo>
+    <gazebo reference="front_left_wheel_link">
+        <material>Gazebo/Purple</material>
+        <mu1 value="${MU1}" />
+        <mu2 value="${MU2}" />
+    </gazebo>
+    <gazebo reference="front_right_wheel_link">
+        <material>Gazebo/Purple</material>
+        <mu1 value="${MU1}" />
+        <mu2 value="${MU2}" />
+    </gazebo>
+    <gazebo reference="back_left_wheel_link">
+        <material>Gazebo/Purple</material>
+        <mu1 value="${MU1}" />
+        <mu2 value="${MU2}" />
+    </gazebo>
+    <gazebo reference="back_right_wheel_link">
+        <material>Gazebo/Purple</material>
+        <mu1 value="${MU1}" />
+        <mu2 value="${MU2}" />
+    </gazebo>
+</robot>
